File: hardware/heater-controller/Thermistor.kicad_sch (KiCad schematic)
At the start: 3 parts, among them J301 Thermistor

Commit message: kicad編集
Parts:
- C301: footprint Capacitor_SMD:C_0402_1005Metric -> Capacitor_SMD:C_0805_2012Metric
Changed lines of the file:
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@@
 			)
 		)
-		(property "Footprint" "Capacitor_SMD:C_0402_1005Metric"
+		(property "Footprint" "Capacitor_SMD:C_0805_2012Metric"
 			(at 145.7452 86.36 0)
 			(effects

Commit message: BBMで問題がなければ発注可能
Parts:
- added C302: 0.1u, Capacitor_SMD:C_0805_2012Metric, symbol Device:C
- added J302: Thermistor2, Connector_JST:JST_PH_B2B-PH-K_1x02_P2.00mm_Vertical, symbol Connector_Generic:Conn_01x02
- added R302: 100k, Resistor_THT:R_Axial_DIN0204_L3.6mm_D1.6mm_P5.08mm_Horizontal, symbol Device:R
- J301: value Thermistor -> Thermistor1
Connections:
- net AGND: now also C302.1, R302.2
- net VDD: now also J302.1 (Pin_1)
- net R_Thermistor renamed R_Thermistor1
- new net R_Thermistor2: C302.2, J302.2 (Pin_2), R302.1
